File: SOURCES/FreeDSP_SMD.sch (KiCad schematic (older format))
At the start: 85 parts, among them IC1 AD8608, IC2 ADAU1701, IC3 24AA256, IC4 TC7SZ08, K1 IN12, K2 OUT34, K3 OUT12, P1 CONN_02X11, P2 CONN_2, P3 CONN_02X02, P4 USBi, P5 CONN_02X13, Q1 PNP, U1 78033, U2 4040, U3 7805, X1 12M288Hz

Commit message: - PLL filter now referenced to +3V3
Connections:
- wire segments 90 -> 88
Other:
- moved on the sheet: C30, C31
Changed lines of the file:
@@
 L C-RESCUE-FreeDSP_SMD C31
 U 1 1 5539768A
-P 8800 4550
-F 0 "C31" H 8800 4650 40  0000 L CNN
-F 1 "56n" H 8806 4465 40  0000 L CNN
-F 2 "Capacitors_SMD:C_0805" H 8838 4400 30  0001 C CNN
-F 3 "~" H 8800 4550 60  0000 C CNN
-	1    8800 4550
-	0    -1   -1   0
+P 8600 4350
+F 0 "C31" H 8600 4450 40  0000 L CNN
+F 1 "56n" H 8606 4265 40  0000 L CNN
+F 2 "Capacitors_SMD:C_0805" H 8638 4200 30  0001 C CNN
+F 3 "~" H 8600 4350 60  0000 C CNN
+	1    8600 4350
+	1    0    0    -1
 $EndComp
 $Comp
 L C-RESCUE-FreeDSP_SMD C30
 U 1 1 55397690
-P 8800 4350
-F 0 "C30" H 8800 4450 40  0000 L CNN
-F 1 "3n3" H 8806 4265 40  0000 L CNN
-F 2 "Capacitors_SMD:C_0805" H 8838 4200 30  0001 C CNN
-F 3 "~" H 8800 4350 60  0000 C CNN
-	1    8800 4350
-	0    -1   -1   0
-$EndComp
-$Comp
-L GND-RESCUE-FreeDSP_SMD #PWR017
-U 1 1 553976AA
-P 9000 4550
-F 0 "#PWR017" H 9000 4550 30  0001 C CNN
-F 1 "GND" H 9000 4480 30  0001 C CNN
-F 2 "" H 9000 4550 60  0000 C CNN
-F 3 "" H 9000 4550 60  0000 C CNN
-	1    9000 4550
-	0    -1   -1   0
-$EndComp
-$Comp
-L GND-RESCUE-FreeDSP_SMD #PWR018
-U 1 1 553976B0
-P 9000 4350
-F 0 "#PWR018" H 9000 4350 30  0001 C CNN
-F 1 "GND" H 9000 4280 30  0001 C CNN
-F 2 "" H 9000 4350 60  0000 C CNN
-F 3 "" H 9000 4350 60  0000 C CNN
-	1    9000 4350
-	0    -1   -1   0
+P 8100 4350
+F 0 "C30" H 8100 4450 40  0000 L CNN
+F 1 "3n3" H 8106 4265 40  0000 L CNN
+F 2 "Capacitors_SMD:C_0805" H 8138 4200 30  0001 C CNN
+F 3 "~" H 8100 4350 60  0000 C CNN
+	1    8100 4350
+	1    0    0    -1
 $EndComp
 $Comp
@@
 	6250 3550 6250 3900
 Connection ~ 8100 4550
-Wire Wire Line
-	8600 4350 8100 4350
-Wire Wire Line
-	8100 4350 8100 4550
 $Comp
 L GND-RESCUE-FreeDSP_SMD #PWR027
@@
 Text GLabel 1550 2850 2    47   Input ~ 0
 MP4
+$Comp
+L 3V3 #PWR?
+U 1 1 56F696D9
+P 8100 4150
+F 0 "#PWR?" H 8100 4250 40  0001 C CNN
+F 1 "3V3" H 8100 4275 40  0000 C CNN
+F 2 "" H 8100 4150 60  0000 C CNN
+F 3 "" H 8100 4150 60  0000 C CNN
+	1    8100 4150
+	1    0    0    -1
+$EndComp
+$Comp
+L 3V3 #PWR?
+U 1 1 56F69AFD
+P 8600 4150
+F 0 "#PWR?" H 8600 4250 40  0001 C CNN
+F 1 "3V3" H 8600 4275 40  0000 C CNN
+F 2 "" H 8600 4150 60  0000 C CNN
+F 3 "" H 8600 4150 60  0000 C CNN
+	1    8600 4150
+	1    0    0    -1
+$EndComp
 $EndSCHEMATC

Commit message: - added pullup for WP Pin
Parts:
- added R28: 10k, Resistors_SMD:R_0805, symbol R-RESCUE-FreeDSP_SMD
Connections:
- wire segments 88 -> 89
Other:
- moved on the sheet: C38, IC3, R24, R25

Commit message: - added selectable LRCLK and BCK bridges for pseudo master mode on inputs - added GERBER folder - added labels
Parts:
- added JP2: LRCLK_BRIDGE, Pin_Headers:Pin_Header_Straight_1x02, symbol JUMPER
- added JP3: BCK_BRIDGE, Pin_Headers:Pin_Header_Straight_1x02, symbol JUMPER
- JP1: value JUMPER -> 5V ext
Changed lines of the file:
@@
 LIBS:contrib
 LIBS:valves
-LIBS:alexlib
 LIBS:FreeDSP_SMD-cache
 EELAYER 25 0
@@
 P 1850 3650
 F 0 "JP1" H 1850 3800 50  0000 C CNN
-F 1 "JUMPER" H 1850 3570 50  0000 C CNN
+F 1 "5V ext" H 1850 3570 50  0000 C CNN
 F 2 "Pin_Headers:Pin_Header_Straight_1x02" H 1850 3650 60  0001 C CNN
 F 3 "" H 1850 3650 60  0000 C CNN
@@
 Wire Wire Line
 	2800 4750 2800 4650
+$Comp
+L JUMPER JP2
+U 1 1 575AD9D5
+P 1300 4100
+F 0 "JP2" H 1300 4250 50  0000 C CNN
+F 1 "LRCLK_BRIDGE" H 1300 4020 50  0000 C CNN
+F 2 "Pin_Headers:Pin_Header_Straight_1x02" H 1300 4100 60  0001 C CNN
+F 3 "" H 1300 4100 60  0000 C CNN
+	1    1300 4100
+	1    0    0    -1
+$EndComp
+$Comp
+L JUMPER JP3
+U 1 1 575ADB7C
+P 1300 4450
+F 0 "JP3" H 1300 4600 50  0000 C CNN
+F 1 "BCK_BRIDGE" H 1300 4370 50  0000 C CNN
+F 2 "Pin_Headers:Pin_Header_Straight_1x02" H 1300 4450 60  0001 C CNN
+F 3 "" H 1300 4450 60  0000 C CNN
+	1    1300 4450
+	1    0    0    -1
+$EndComp
+Text GLabel 1000 4100 0    47   Input ~ 0
+MP4
+Text GLabel 1600 4100 2    47   Input ~ 0
+MP10
+Text GLabel 1000 4450 0    47   Input ~ 0
+MP5
+Text GLabel 1600 4450 2    47   Input ~ 0
+MP11
 $EndSCHEMATC

Commit message: + added GERBER folder + WP jumper for EEPROM flashing ~ I2C pullups reduced to 1k5 (400khz selfboot needs faster risetimes) ~ Reset pullup reduced to 4k7 (DAC board has 10k pulldown onboard) ~ incremented version to 1.1
Parts:
- removed Q1: PNP, Housings_SOT-23_SOT-143_TSOT-6:SOT-23, symbol PNP
- added JP4: WP, Pin_Headers:Pin_Header_Straight_1x02_Pitch2.54mm, symbol JUMPER
- added Q1: Q_PNP_BEC, TO_SOT_Packages_SMD:SOT-23, symbol Q_PNP_BEC
- JP1, JP2, JP3: footprint Pin_Headers:Pin_Header_Straight_1x02 -> Pin_Headers:Pin_Header_Straight_1x02_Pitch2.54mm
- R24, R25: value 10k -> 1k5
- R9: value 18k -> 4k7
Connections:
- wire segments 89 -> 90
Other:
- note removed: "<= 1% Toleranze"
- moved on the sheet: C38, IC3, R24, R25, R28
Changed lines of the file:
@@
 P 4050 3250
 F 0 "R9" V 4130 3250 40  0000 C CNN
-F 1 "18k" V 4057 3251 40  0000 C CNN
+F 1 "4k7" V 4057 3251 40  0000 C CNN
 F 2 "Resistors_SMD:R_0805" V 3980 3250 30  0001 C CNN
 F 3 "~" H 4050 3250 30  0000 C CNN
@@
 Text Label 5850 6100 3    60   ~ 0
 MP10
-$Comp
-L PNP Q1
-U 1 1 553971F3
-P 5950 6750
-F 0 "Q1" H 5950 6600 60  0000 R CNN
-F 1 "PNP" H 5950 6900 60  0000 R CNN
-F 2 "Housings_SOT-23_SOT-143_TSOT-6:SOT-23" H 5950 6750 60  0001 C CNN
-F 3 "~" H 5950 6750 60  0000 C CNN
-	1    5950 6750
-	0    -1   1    0
-$EndComp
 $Comp
 L 3V3 #PWR07
@@
 L I2CFLASH IC3
 U 1 1 5539B417
-P 10400 5850
-F 0 "IC3" H 10400 5850 60  0000 C CNN
-F 1 "24AA256" H 10400 6150 60  0000 C CNN
-F 2 "Housings_SOIC:SOIC-8_3.9x4.9mm_Pitch1.27mm" H 10400 5850 60  0001 C CNN
-F 3 "" H 10400 5850 60  0000 C CNN
-	1    10400 5850
+P 10400 5650
+F 0 "IC3" H 10400 5650 60  0000 C CNN
+F 1 "24AA256" H 10400 5950 60  0000 C CNN
+F 2 "Housings_SOIC:SOIC-8_3.9x4.9mm_Pitch1.27mm" H 10400 5650 60  0001 C CNN
+F 3 "" H 10400 5650 60  0000 C CNN
+	1    10400 5650
 	-1   0    0    -1
 $EndComp
@@
 L C-RESCUE-FreeDSP_SMD C38
 U 1 1 5539B42A
-P 9850 5500
-F 0 "C38" H 9850 5600 40  0000 L CNN
-F 1 "100n" H 9856 5415 40  0000 L CNN
-F 2 "Capacitors_SMD:C_0805" H 9888 5350 30  0001 C CNN
-F 3 "~" H 9850 5500 60  0000 C CNN
-	1    9850 5500
+P 9850 5300
+F 0 "C38" H 9850 5400 40  0000 L CNN
+F 1 "100n" H 9856 5215 40  0000 L CNN
+F 2 "Capacitors_SMD:C_0805" H 9888 5150 30  0001 C CNN
+F 3 "~" H 9850 5300 60  0000 C CNN
+	1    9850 5300
 	-1   0    0    1
 $EndComp
@@
 L GND-RESCUE-FreeDSP_SMD #PWR057
 U 1 1 5539B43A
-P 10950 6000
-F 0 "#PWR057" H 10950 6000 30  0001 C CNN
-F 1 "GND" H 10950 5930 30  0001 C CNN
-F 2 "" H 10950 6000 60  0000 C CNN
-F 3 "" H 10950 6000 60  0000 C CNN
-	1    10950 6000
-	0    -1   -1   0
-$EndComp
-$Comp
-L GND-RESCUE-FreeDSP_SMD #PWR058
-U 1 1 5539B440
-P 9850 5300
-F 0 "#PWR058" H 9850 5300 30  0001 C CNN
-F 1 "GND" H 9850 5230 30  0001 C CNN
-F 2 "" H 9850 5300 60  0000 C CNN
-F 3 "" H 9850 5300 60  0000 C CNN
-	1    9850 5300
-	-1   0    0    1
-$EndComp
-$Comp
-L 3V3 #PWR059
-U 1 1 5539B446
-P 9850 5700
-F 0 "#PWR059" H 9850 5800 40  0001 C CNN
-F 1 "3V3" H 9850 5825 40  0000 C CNN
-F 2 "" H 9850 5700 60  0000 C CNN
-F 3 "" H 9850 5700 60  0000 C CNN
-	1    9850 5700
-	0    -1   1    0
-$EndComp
-$Comp
-L GND-RESCUE-FreeDSP_SMD #PWR060
-U 1 1 5539B57E
-P 10950 5900
-F 0 "#PWR060" H 10950 5900 30  0001 C CNN
-F 1 "GND" H 10950 5830 30  0001 C CNN
-F 2 "" H 10950 5900 60  0000 C CNN
-F 3 "" H 10950 5900 60  0000 C CNN
-	1    10950 5900
-	0    -1   -1   0
-$EndComp
-$Comp
-L GND-RESCUE-FreeDSP_SMD #PWR061
-U 1 1 5539B584
 P 10950 5800
-F 0 "#PWR061" H 10950 5800 30  0001 C CNN
+F 0 "#PWR057" H 10950 5800 30  0001 C CNN
 F 1 "GND" H 10950 5730 30  0001 C CNN
 F 2 "" H 10950 5800 60  0000 C CNN
@@
 $EndComp
 $Comp
-L GND-RESCUE-FreeDSP_SMD #PWR062
-U 1 1 5539B58A
+L GND-RESCUE-FreeDSP_SMD #PWR058
+U 1 1 5539B440
+P 9850 5100
+F 0 "#PWR058" H 9850 5100 30  0001 C CNN
+F 1 "GND" H 9850 5030 30  0001 C CNN
+F 2 "" H 9850 5100 60  0000 C CNN
+F 3 "" H 9850 5100 60  0000 C CNN
+	1    9850 5100
+	-1   0    0    1
+$EndComp
+$Comp
+L 3V3 #PWR059
+U 1 1 5539B446
+P 9850 5500
+F 0 "#PWR059" H 9850 5600 40  0001 C CNN
+F 1 "3V3" H 9850 5625 40  0000 C CNN
+F 2 "" H 9850 5500 60  0000 C CNN
+F 3 "" H 9850 5500 60  0000 C CNN
+	1    9850 5500
+	0    -1   1    0
+$EndComp
+$Comp
+L GND-RESCUE-FreeDSP_SMD #PWR060
+U 1 1 5539B57E
 P 10950 5700
-F 0 "#PWR062" H 10950 5700 30  0001 C CNN
+F 0 "#PWR060" H 10950 5700 30  0001 C CNN
 F 1 "GND" H 10950 5630 30  0001 C CNN
 F 2 "" H 10950 5700 60  0000 C CNN
@@
 $EndComp
 $Comp
+L GND-RESCUE-FreeDSP_SMD #PWR061
+U 1 1 5539B584
+P 10950 5600
+F 0 "#PWR061" H 10950 5600 30  0001 C CNN
+F 1 "GND" H 10950 5530 30  0001 C CNN
+F 2 "" H 10950 5600 60  0000 C CNN
+F 3 "" H 10950 5600 60  0000 C CNN
+	1    10950 5600
+	0    -1   -1   0
+$EndComp
+$Comp
+L GND-RESCUE-FreeDSP_SMD #PWR062
+U 1 1 5539B58A
+P 10950 5500
+F 0 "#PWR062" H 10950 5500 30  0001 C CNN
+F 1 "GND" H 10950 5430 30  0001 C CNN
+F 2 "" H 10950 5500 60  0000 C CNN
+F 3 "" H 10950 5500 60  0000 C CNN
+	1    10950 5500
+	0    -1   -1   0
+$EndComp
+$Comp
 L R-RESCUE-FreeDSP_SMD R25
 U 1 1 5539B590
-P 9400 5550
-F 0 "R25" V 9480 5550 40  0000 C CNN
-F 1 "10k" V 9407 5551 40  0000 C CNN
-F 2 "Resistors_SMD:R_0805" V 9330 5550 30  0001 C CNN
-F 3 "~" H 9400 5550 30  0000 C CNN
-	1    9400 5550
+P 9400 5350
+F 0 "R25" V 9480 5350 40  0000 C CNN
+F 1 "1k5" V 9407 5351 40  0000 C CNN
+F 2 "Resistors_SMD:R_0805" V 9330 5350 30  0001 C CNN
+F 3 "~" H 9400 5350 30  0000 C CNN
+	1    9400 5350
 	1    0    0    1
 $EndComp
@@
 L R-RESCUE-FreeDSP_SMD R24
 U 1 1 5539B596
-P 9250 5550
-F 0 "R24" V 9330 5550 40  0000 C CNN
-F 1 "10k" V 9257 5551 40  0000 C CNN
-F 2 "Resistors_SMD:R_0805" V 9180 5550 30  0001 C CNN
-F 3 "~" H 9250 5550 30  0000 C CNN
-	1    9250 5550
+P 9250 5350
+F 0 "R24" V 9330 5350 40  0000 C CNN
+F 1 "1k5" V 9257 5351 40  0000 C CNN
+F 2 "Resistors_SMD:R_0805" V 9180 5350 30  0001 C CNN
+F 3 "~" H 9250 5350 30  0000 C CNN
+	1    9250 5350
 	1    0    0    1
 $EndComp
@@
 L 3V3 #PWR063
 U 1 1 5539B693
-P 9400 5300
-F 0 "#PWR063" H 9400 5400 40  0001 C CNN
-F 1 "3V3" H 9400 5425 40  0000 C CNN
-F 2 "" H 9400 5300 60  0000 C CNN
-F 3 "" H 9400 5300 60  0000 C CNN
-	1    9400 5300
+P 9400 5100
+F 0 "#PWR063" H 9400 5200 40  0001 C CNN
+F 1 "3V3" H 9400 5225 40  0000 C CNN
+F 2 "" H 9400 5100 60  0000 C CNN
+F 3 "" H 9400 5100 60  0000 C CNN
+	1    9400 5100
 	-1   0    0    -1
 $EndComp
@@
 L 3V3 #PWR064
 U 1 1 5539B699
-P 9250 5300
-F 0 "#PWR064" H 9250 5400 40  0001 C CNN
-F 1 "3V3" H 9250 5425 40  0000 C CNN
-F 2 "" H 9250 5300 60  0000 C CNN
-F 3 "" H 9250 5300 60  0000 C CNN
-	1    9250 5300
+P 9250 5100
+F 0 "#PWR064" H 9250 5200 40  0001 C CNN
+F 1 "3V3" H 9250 5225 40  0000 C CNN
+F 2 "" H 9250 5100 60  0000 C CNN
+F 3 "" H 9250 5100 60  0000 C CNN
+	1    9250 5100
 	-1   0    0    -1
 $EndComp
-Text Label 9250 6000 2    60   ~ 0
+Text Label 9250 5800 2    60   ~ 0
 SDA
-Text Label 9400 5900 2    60   ~ 0
+Text Label 9400 5700 2    60   ~ 0
 SCL
 $Comp
@@
 Text Label 10750 4850 0    60   ~ 0
 MCLK
-Text Label 9550 5800 2    60   ~ 0
+Text Label 9550 5600 2    60   ~ 0
 WP
-Text Notes 6400 6550 0    60   ~ 0
-<= 1% Toleranze
 Text Notes 4300 4600 1    60   ~ 0
 <=1%
@@
 F 0 "JP1" H 1850 3800 50  0000 C CNN
 F 1 "5V ext" H 1850 3570 50  0000 C CNN
-F 2 "Pin_Headers:Pin_Header_Straight_1x02" H 1850 3650 60  0001 C CNN
+F 2 "Pin_Headers:Pin_Header_Straight_1x02_Pitch2.54mm" H 1850 3650 60  0001 C CNN
 F 3 "" H 1850 3650 60  0000 C CNN
 	1    1850 3650
@@
 L R-RESCUE-FreeDSP_SMD R28
 U 1 1 573ADFB1
-P 9550 5550
-F 0 "R28" V 9630 5550 40  0000 C CNN
-F 1 "10k" V 9557 5551 40  0000 C CNN
-F 2 "Resistors_SMD:R_0805" V 9480 5550 30  0001 C CNN
-F 3 "~" H 9550 5550 30  0000 C CNN
-	1    9550 5550
+P 9550 5350
+F 0 "R28" V 9630 5350 40  0000 C CNN
+F 1 "10k" V 9557 5351 40  0000 C CNN
+F 2 "Resistors_SMD:R_0805" V 9480 5350 30  0001 C CNN
+F 3 "~" H 9550 5350 30  0000 C CNN
+	1    9550 5350
 	1    0    0    1
 $EndComp
@@
 L 3V3 #PWR084
 U 1 1 573AE413
-P 9550 5300
-F 0 "#PWR084" H 9550 5400 40  0001 C CNN
-F 1 "3V3" H 9550 5425 40  0000 C CNN
-F 2 "" H 9550 5300 60  0000 C CNN
-F 3 "" H 9550 5300 60  0000 C CNN
-	1    9550 5300
+P 9550 5100
+F 0 "#PWR084" H 9550 5200 40  0001 C CNN
+F 1 "3V3" H 9550 5225 40  0000 C CNN
+F 2 "" H 9550 5100 60  0000 C CNN
+F 3 "" H 9550 5100 60  0000 C CNN
+	1    9550 5100
 	-1   0    0    -1
 $EndComp
@@
 	4050 3500 4050 4950
 Connection ~ 4050 4850
-Connection ~ 9850 5700
-Wire Wire Line
-	9400 5800 9400 5900
-Wire Wire Line
-	9400 5900 9850 5900
-Wire Wire Line
-	9850 6000 9250 6000
-Wire Wire Line
-	9250 6000 9250 5800
+Connection ~ 9850 5500
+Wire Wire Line
+	9400 5600 9400 5700
+Wire Wire Line
+	9400 5700 9850 5700
+Wire Wire Line
+	9850 5800 9250 5800
+Wire Wire Line
+	9250 5800 9250 5600
 Connection ~ 4050 3500
 Wire Wire Line
@@
 Connection ~ 9250 3050
 Wire Wire Line
-	9850 5800 9550 5800
+	9850 5600 9550 5600
 Wire Wire Line
 	2800 4750 2800 4650
@@
 F 0 "JP2" H 1300 4250 50  0000 C CNN
 F 1 "LRCLK_BRIDGE" H 1300 4020 50  0000 C CNN
-F 2 "Pin_Headers:Pin_Header_Straight_1x02" H 1300 4100 60  0001 C CNN
+F 2 "Pin_Headers:Pin_Header_Straight_1x02_Pitch2.54mm" H 1300 4100 60  0001 C CNN
 F 3 "" H 1300 4100 60  0000 C CNN
 	1    1300 4100
@@
 F 0 "JP3" H 1300 4600 50  0000 C CNN
 F 1 "BCK_BRIDGE" H 1300 4370 50  0000 C CNN
-F 2 "Pin_Headers:Pin_Header_Straight_1x02" H 1300 4450 60  0001 C CNN
+F 2 "Pin_Headers:Pin_Header_Straight_1x02_Pitch2.54mm" H 1300 4450 60  0001 C CNN
 F 3 "" H 1300 4450 60  0000 C CNN
 	1    1300 4450
@@
 Text GLabel 1600 4450 2    47   Input ~ 0
 MP11
+$Comp
+L JUMPER JP4
+U 1 1 59DD976C
+P 9550 6150
+F 0 "JP4" H 9550 6300 50  0000 C CNN
+F 1 "WP" H 9550 6070 50  0000 C CNN
+F 2 "Pin_Headers:Pin_Header_Straight_1x02_Pitch2.54mm" H 9550 6150 60  0001 C CNN
+F 3 "" H 9550 6150 60  0000 C CNN
+	1    9550 6150
+	0    1    1    0
+$EndComp
+Wire Wire Line
+	9550 5600 9550 5850
+Connection ~ 9550 5600
+$Comp
+L GND-RESCUE-FreeDSP_SMD #PWR085
+U 1 1 59DDC992
+P 9550 6450
+F 0 "#PWR085" H 9550 6450 30  0001 C CNN
+F 1 "GND" H 9550 6380 30  0001 C CNN
+F 2 "" H 9550 6450 60  0000 C CNN
+F 3 "" H 9550 6450 60  0000 C CNN
+	1    9550 6450
+	1    0    0    -1
+$EndComp
+$Comp
+L Q_PNP_BEC Q1
+U 1 1 59DE7822
+P 5950 6750
+F 0 "Q1" H 6250 6800 50  0000 R CNN
+F 1 "Q_PNP_BEC" H 6550 6700 50  0000 R CNN
+F 2 "TO_SOT_Packages_SMD:SOT-23" H 6150 6850 50  0001 C CNN
+F 3 "" H 5950 6750 50  0000 C CNN
+	1    5950 6750
+	0    -1   1    0
+$EndComp
 $EndSCHEMATC

Commit message: - migrated to KiCAD 5
Parts:
- C1, C10, C11, C12, C13, C14, C15, C16, C17, C18, C19, C2, C20, C21, C22, C23, C24, C25, C26, C27, C28, C29, C3, C30, C31, C32, C33, C34, C35, C36, C37, C38, C39, C40, C5, C6, C7, C9: symbol C-RESCUE-FreeDSP_SMD -> FreeDSP_SMD-rescue:C-RESCUE-FreeDSP_SMD
- C4, C8: symbol CAPAPOL -> FreeDSP_SMD-rescue:CAPAPOL
- IC1: symbol OPAMP4 -> FreeDSP_SMD-rescue:OPAMP4
- IC2: symbol ADAU1701 -> FreeDSP_SMD-rescue:ADAU1701
- IC3: symbol I2CFLASH -> FreeDSP_SMD-rescue:I2CFLASH
- IC4: symbol TC7SZ08 -> FreeDSP_SMD-rescue:TC7SZ08
- JP1, JP2, JP3, JP4: symbol JUMPER -> FreeDSP_SMD-rescue:JUMPER
- K1, K2, K3: symbol CONN_3 -> FreeDSP_SMD-rescue:CONN_3
- P1: symbol CONN_02X11 -> FreeDSP_SMD-rescue:CONN_02X11
- P2: symbol CONN_2 -> FreeDSP_SMD-rescue:CONN_2
- P3: symbol CONN_02X02 -> FreeDSP_SMD-rescue:CONN_02X02
- P4: symbol CONN_10 -> FreeDSP_SMD-rescue:CONN_10
- P5: symbol CONN_02X13 -> FreeDSP_SMD-rescue:CONN_02X13
- Q1: symbol Q_PNP_BEC -> Device:Q_PNP_BEC
- R1, R10, R11, R12, R13, R14, R15, R16, R17, R18, R19, R2, R20, R21, R22, R23, R24, R25, R26, R27, R28, R3, R4, R5, R6, R7, R8, R9: symbol R-RESCUE-FreeDSP_SMD -> FreeDSP_SMD-rescue:R-RESCUE-FreeDSP_SMD
- U1, U3: symbol 7805 -> FreeDSP_SMD-rescue:7805
- U2: symbol 4040 -> cmos4000:4040
- X1: symbol CRYSTAL -> FreeDSP_SMD-rescue:CRYSTAL
Connections:
- wire segments 90 -> 131

Commit message: - fixed a missing track
Parts:
- U2: symbol cmos4000:4040 -> FreeDSP_SMD-rescue:4040-cmos4000
Changed lines of the file:
@@
 _RESET
 $Comp
-L cmos4000:4040 U2
+L FreeDSP_SMD-rescue:4040-cmos4000 U2
 U 1 1 5664C8DB
 P 9900 3850
